Commit message: updated

File: mir1350v5_1_description/urdf/mir1350v5_1.xacro (robot description, xacro)
@@ -666,5 +666,6 @@
   <parent link="abb_link5__1__1"/>
   <child link="abb_link6__1__1"/>
-  <axis xyz="0.011956 0.999883 -0.009509"/>
+  <!-- <axis xyz="0.011956 0.999883 -0.009509"/> -->
+  <axis xyz="-0.011956 0.999883 0.009509"/>
   <!-- <limit effort="1000" lower="-2.181" upper="2.094" velocity="4.363"/> -->
   <limit effort="1000" lower="0" upper="2.094" velocity="4.363"/>
@@ -680,5 +681,5 @@
   <parent link="abb_link6__1__1"/>
   <child link="abb_link7__4__1"/>
-  <axis xyz="0.999586 0.011703 0.026282"/>
+  <axis xyz="-0.999586 0.011703 0.026282"/>
   <!-- <limit effort="1000" lower="-6.981" upper="6.981" velocity="6.283"/> -->
   <limit effort="1000" lower="0" upper="6.981" velocity="6.283"/>
@@ -695,4 +696,5 @@
   <child link="box__1__1"/>
 </joint>
+<!-- Wheel joints -->
 <joint name="driveWheelRight_fixedJoint" type="continuous">
   <origin xyz="0.0 0.3553 0.0565" rpy="0 0 0"/>
@@ -707,3 +709,4 @@
   <axis xyz="0.0 -1.0 0.0"/>
 </joint>
+<!--End of  "Wheel joints" -->
 </robot>

Commit message: roslaunch mir1350v5_1_description run_all.launch

File: mir1350v5_1_description/urdf/mir1350v5_1.xacro (robot description, xacro)
@@ -612,5 +612,5 @@
   <axis xyz="0.0 -0.0 1.0"/>
   <!-- <limit effort="1000" lower="-3.141" upper="3.141" velocity="3.054"/> -->
-  <limit effort="1000" lower="0" upper="3.141" velocity="3.054"/>
+  <limit effort="1000" lower="-3.141" upper="3.141" velocity="3.054"/>
 </joint>
 <!-- <joint name="abbLink3_revJoint" type="continuous">
@@ -626,5 +626,5 @@
   <axis xyz="0.011845 -0.99993 -0.0"/>
   <!-- <limit effort="1000" lower="-1.570" upper="2.617" velocity="3.054"/> -->
-  <limit effort="1000" lower="0" upper="2.617" velocity="3.054"/>
+  <limit effort="1000" lower="-3.141" upper="3.141" velocity="3.054"/>
 </joint>
 <!-- <joint name="abbLink4_revJoint" type="continuous">
@@ -640,5 +640,5 @@
   <axis xyz="-0.011845 -0.99993 0.0"/>
   <!-- <limit effort="1000" lower="-3.141" upper="1.308" velocity="3.054"/> -->
-  <limit effort="1000" lower="0" upper="1.308" velocity="3.054"/>
+  <limit effort="1000" lower="-3.141" upper="3.141" velocity="3.054"/>
 </joint>
 <!-- <joint name="abbLink5_revJoint" type="continuous">
@@ -654,5 +654,5 @@
   <axis xyz="0.999861 0.011844 0.011753"/>
   <!-- <limit effort="1000" lower="-6.981" upper="6.981" velocity="4.363"/> -->
-  <limit effort="1000" lower="0" upper="6.981" velocity="4.363"/>
+  <limit effort="1000" lower="-3.141" upper="3.141" velocity="3.054"/>
 </joint>
 <!-- <joint name="abbLink6_revJoint" type="continuous">
@@ -669,5 +669,5 @@
   <axis xyz="-0.011956 0.999883 0.009509"/>
   <!-- <limit effort="1000" lower="-2.181" upper="2.094" velocity="4.363"/> -->
-  <limit effort="1000" lower="0" upper="2.094" velocity="4.363"/>
+  <limit effort="1000" lower="-3.141" upper="3.141" velocity="3.054"/>
 </joint>
 <!-- <joint name="abbLink7_revJoint" type="continuous">
